File: Board/Kicad/SmartIRClip.kicad_pcb (KiCad board)
At the start: 4 copper layers, 47.5 x 48 mm, 72 parts, among them J1 USB_OTG, Q1 DMP1045U, Q2 BC817-40, Q3 BC807-40, Q4 DMP1045U, U1 MCP73832, U2 MSP430FR2433, U3 MCP1700T, U4 FT232RL, U5 LSM303AGRTR

Commit message: cleanup
Parts:
- moved R17 2.20 mm to (92.2, 93.7), turned to 0 degrees
Connections:
- U2 pad : GND -> (no net)
Routing:
- net GND: track 10.6 -> 23.7 mm
- net /BRIGHT+_SW: track 58.4 -> 67.6 mm
- net /USB_VCC: track 57.1 -> 61.8 mm
- net Net-(BT1-Pad1): track 32.0 -> 33.1 mm
- net /INT_2_XL: track 12.9 -> 12.1 mm
- net Net-(Q2-Pad3): track 7.38 -> 6.78 mm

Commit message: more cleanup
Routing:
- net GND: track 23.7 -> 28.6 mm
Changed lines of the file:
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@@
     (thickness 1.6)
     (drawings 24)
-    (tracks 516)
+    (tracks 521)
     (zones 0)
     (modules 72)
@@
   (via (at 86.225 63) (size 0.7) (drill 0.35) (layers Top_Copper Bottom_Copper) (net 1))
   (via (at 82.625 68.075) (size 0.7) (drill 0.35) (layers Top_Copper Bottom_Copper) (net 1))
+  (segment (start 72.5 70.8) (end 73.429 70.8) (width 0.254) (layer Top_Copper) (net 2))
+  (segment (start 73.429 70.8) (end 73.729 70.5) (width 0.254) (layer Top_Copper) (net 2))
+  (segment (start 72.5 70.15) (end 73.429 70.15) (width 0.254) (layer Top_Copper) (net 2))
+  (segment (start 73.429 70.15) (end 73.779 70.5) (width 0.254) (layer Top_Copper) (net 2))
+  (segment (start 74.4 81.475) (end 76.475 81.475) (width 0.254) (layer Top_Copper) (net 2))
   (segment (start 74.4 84.075) (end 73.075 84.075) (width 0.254) (layer Top_Copper) (net 2))
   (segment (start 74.4 84.725) (end 72.775 84.725) (width 0.254) (layer Top_Copper) (net 2))
