File: Board/Kicad/SmartIRClip.kicad_pcb (KiCad board)
At the start: 4 copper layers, 47.5 x 48 mm, 72 parts, among them J1 USB_OTG, Q1 DMP1045U, Q2 BC817-40, Q3 BC807-40, Q4 DMP1045U, U1 MCP73832, U2 MSP430FR2433, U3 MCP1700T, U4 FT232RL, U5 LSM303AGRTR

Commit message: cleanup
Routing:
- net /USB_IN_SENSE: track 21.4 -> 26.4 mm
- net /XL_SCL: track 13.4 -> 14.6 mm
Changed lines of the file:
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@@
     (thickness 1.6)
     (drawings 24)
-    (tracks 520)
+    (tracks 522)
     (zones 0)
     (modules 72)
@@
   (via (at 93.472 82.804) (size 0.7) (drill 0.35) (layers Top_Copper Bottom_Copper) (net 27))
   (segment (start 87.26 74.53) (end 87.26 76.03) (width 0.1524) (layer Top_Copper) (net 27) (status 30))
-  (segment (start 94.996 68.326) (end 95.345999 68.675999) (width 0.1524) (layer Bottom_Copper) (net 28))
+  (segment (start 91 67.1) (end 91.6024 67.1) (width 0.1524) (layer Top_Copper) (net 28))
+  (segment (start 92.8284 68.326) (end 94.501026 68.326) (width 0.1524) (layer Top_Copper) (net 28))
+  (segment (start 91.6024 67.1) (end 92.8284 68.326) (width 0.1524) (layer Top_Copper) (net 28))
+  (segment (start 94.501026 68.326) (end 94.996 68.326) (width 0.1524) (layer Top_Copper) (net 28))
+  (segment (start 94.996 68.326) (end 95.834934 68.326) (width 0.1524) (layer Bottom_Copper) (net 28))
+  (segment (start 95.834934 68.326) (end 99.77119 72.262256) (width 0.1524) (layer Bottom_Copper) (net 28))
   (segment (start 99.481337 74.585597) (end 98.044 74.585597) (width 0.1524) (layer Bottom_Copper) (net 28))
-  (segment (start 95.345999 68.675999) (end 96.184933 68.675999) (width 0.1524) (layer Bottom_Copper) (net 28))
   (segment (start 96.184933 68.675999) (end 99.77119 72.262256) (width 0.1524) (layer Bottom_Copper) (net 28))
   (segment (start 99.77119 72.262256) (end 99.77119 74.295744) (width 0.1524) (layer Bottom_Copper) (net 28))
@@
   (via (at 98.044 74.585597) (size 0.7) (drill 0.35) (layers Top_Copper Bottom_Copper) (net 28))
   (segment (start 94.996 77.2415) (end 94.95 77.2875) (width 0.1524) (layer Top_Copper) (net 28) (status 30))
-  (segment (start 91 67.1) (end 91 67.25) (width 0.1524) (layer Top_Copper) (net 28) (status 30))
-  (segment (start 91 67.25) (end 92.076 68.326) (width 0.1524) (layer Top_Copper) (net 28) (status 10))
-  (segment (start 92.076 68.326) (end 94.996 68.326) (width 0.1524) (layer Top_Copper) (net 28))
   (segment (start 89 67.09) (end 90.99 67.09) (width 0.1524) (layer Top_Copper) (net 28) (status 30))
   (segment (start 90.99 67.09) (end 91 67.1) (width 0.1524) (layer Top_Copper) (net 28) (status 30))
@@
   (segment (start 93.95 82.283209) (end 93.95 81.1125) (width 0.1524) (layer Top_Copper) (net 33) (status 20))
   (via (at 94.470791 82.804) (size 0.7) (drill 0.35) (layers Top_Copper Bottom_Copper) (net 33))
+  (segment (start 93.567999 86.275935) (end 94.443934 85.4) (width 0.1524) (layer Internal_1) (net 34))
+  (segment (start 94.443934 85.4) (end 94.601554 85.24238) (width 0.1524) (layer Internal_1) (net 34))
+  (segment (start 93.218 87.122) (end 93.218 86.625934) (width 0.1524) (layer Internal_1) (net 34))
+  (segment (start 93.218 86.625934) (end 94.443934 85.4) (width 0.1524) (layer Internal_1) (net 34))
   (segment (start 89.629602 85.36858) (end 91.46458 85.36858) (width 0.1524) (layer Top_Copper) (net 34) (status 10))
   (segment (start 91.46458 85.36858) (end 93.218 87.122) (width 0.1524) (layer Top_Copper) (net 34))
@@
   (segment (start 95.323194 85.076806) (end 95.323194 82.804) (width 0.1524) (layer Internal_1) (net 34))
   (segment (start 94.601554 85.24238) (end 95.15762 85.24238) (width 0.1524) (layer Internal_1) (net 34))
-  (segment (start 93.218 87.122) (end 93.567999 86.772001) (width 0.1524) (layer Internal_1) (net 34))
-  (segment (start 93.567999 86.275935) (end 94.601554 85.24238) (width 0.1524) (layer Internal_1) (net 34))
-  (segment (start 93.567999 86.772001) (end 93.567999 86.275935) (width 0.1524) (layer Internal_1) (net 34))
   (segment (start 93.5 88.5) (end 93.5 87.404) (width 0.1524) (layer Top_Copper) (net 34) (status 10))
   (segment (start 93.5 87.404) (end 93.218 87.122) (width 0.1524) (layer Top_Copper) (net 34))

Commit message: layer counter
Other:
- board text added: "1"
- board text added: "2"
- board text added: "3"
- board text added: "4"
Changed lines of the file:
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@@
     (area 66.924999 58.924999 114.575001 107.075001)
     (thickness 1.6)
-    (drawings 24)
+    (drawings 28)
     (tracks 522)
     (zones 0)
@@
       (xy 0.555814 -2.531069)) (layer F.SilkS) (width 0.01))
   )
+  (gr_text 4 (at 82.3 105.6) (layer Bottom_Copper)
+    (effects (font (size 1.5 1.5) (thickness 0.3)))
+  )
+  (gr_text 3 (at 80.1 105.6) (layer Internal_2)
+    (effects (font (size 1.5 1.5) (thickness 0.3)))
+  )
+  (gr_text 2 (at 77.8 105.6) (layer Internal_1)
+    (effects (font (size 1.5 1.5) (thickness 0.3)))
+  )
+  (gr_text 1 (at 75.7 105.6) (layer Top_Copper)
+    (effects (font (size 1.5 1.5) (thickness 0.3)))
+  )
   (gr_line (start 108.97 103.16) (end 108.63 102.83) (layer F.SilkS) (width 0.2))

Commit message: board send
Parts:
- moved C14 7.26 mm to (81.3, 88.2)
- moved R10 2.41 mm to (77.9, 74.1)
- moved R11 2.41 mm to (76.3, 74.1)
Routing:
- net +2V5: track 53.5 -> 58.1 mm
- net /USB_D-: track 16.3 -> 13.3 mm
- net /UART_RX: track 9.09 -> 8.92 mm, vias 2 -> 0
