File: Board/Kicad/SmartIRClip.sch (KiCad schematic (older format))
At the start: 66 parts, among them J1 USB_OTG, J2 UART, J3 SPYBYWIRE, Q1 DMP1045U, Q2 BC817-40, Q3 BC807-40, Q4 DMP1045U, SW1 ON/OFF, SW2 BRIGHT+, SW3 BRIGHT-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

Commit message: board send
Parts:
- R13, R14: value 20R -> 40R
- R15, R16: value 10k -> 40R
